File: hardware/annoy-o-tron.brd (EAGLE design)
At the start: 63 x 47.5 mm, 25 parts, among them IC1 TPS61201, J1 DM3AT-SF-PEJM5, Q1 8MHz, U1 ATMEGA328P-AU

Commit message: Fixed for board.
Parts:
- flipped JP1 to the top, turned to 0 degrees
Routing:
- net RESET: track 43.0 -> 41.8 mm
- net GND: track 166.1 -> 165.5 mm
- net VCC/2: vias 1 -> 0
Changed lines of the file:
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@@
 <element name="R1" library="rcl" package="R0805" value="10k" x="37" y="34.5" rot="MR90"/>
 <element name="C13" library="rcl" package="153CLV-0405" value="100uF" x="44" y="11.5" rot="MR270"/>
-<element name="JP1" library="pinhead" package="1X02" value="" x="21" y="45" locked="yes" rot="MR180"/>
+<element name="JP1" library="pinhead" package="1X02" value="" x="21" y="45" locked="yes"/>
 <element name="J1" library="DM3AT-SF-PEJM5" package="DM3AT-SF-PEJM5" value="DM3AT-SF-PEJM5" x="13" y="16.5" locked="yes" rot="MR0"/>
 <element name="JP2" library="avr-7" package="AVR-ISP-6" value="AVR-ISP-6VERT" x="2.5" y="23.75" locked="yes" rot="MR90"/>
@@
 <wire x1="34" y1="7" x2="43" y2="16" width="0.6096" layer="1"/>
 <wire x1="43" y1="16" x2="44" y2="16" width="0.6096" layer="1"/>
-<wire x1="27.2582" y1="24.1564" x2="25.8436" y2="24.1564" width="0.254" layer="16"/>
-<wire x1="25.8436" y1="24.1564" x2="24" y2="26" width="0.254" layer="16"/>
-<wire x1="24" y1="26" x2="21.5" y2="26" width="0.254" layer="16"/>
-<wire x1="21.5" y1="26" x2="20.5" y2="25" width="0.254" layer="16"/>
+<wire x1="27.2582" y1="24.1564" x2="25.8436" y2="24.1564" width="0.4064" layer="16"/>
+<wire x1="25.8436" y1="24.1564" x2="24" y2="26" width="0.4064" layer="16"/>
+<wire x1="24" y1="26" x2="21.5" y2="26" width="0.4064" layer="16"/>
+<wire x1="21.5" y1="26" x2="20.5" y2="25" width="0.4064" layer="16"/>
 <wire x1="18" y1="29.525" x2="17.5" y2="29.525" width="0.254" layer="16"/>
 <wire x1="18" y1="29.525" x2="18" y2="30.725" width="0.254" layer="16"/>
@@
 <wire x1="22" y1="30.5" x2="21.775" y2="30.725" width="0.254" layer="16"/>
 <wire x1="21.775" y1="30.725" x2="18" y2="30.725" width="0.254" layer="16"/>
-<wire x1="19" y1="26" x2="21.5" y2="26" width="0.254" layer="16"/>
-<wire x1="19" y1="26" x2="18" y2="27" width="0.254" layer="16"/>
-<wire x1="18" y1="27" x2="18" y2="29.525" width="0.254" layer="16"/>
-<wire x1="3.77" y1="26.29" x2="6.29" y2="26.29" width="0.6096" layer="1"/>
-<via x="7" y="27" extent="1-16" drill="0.8" diameter="1.6"/>
-<wire x1="7" y1="27" x2="8.5" y2="27" width="0.6096" layer="16"/>
-<wire x1="8.5" y1="27" x2="9" y2="27.5" width="0.6096" layer="16"/>
-<wire x1="9" y1="27.5" x2="9" y2="28.5" width="0.6096" layer="16"/>
-<wire x1="6.29" y1="26.29" x2="7" y2="27" width="0.6096" layer="1"/>
-<wire x1="18.5" y1="32.475" x2="18.5" y2="41" width="0.254" layer="16"/>
-<wire x1="18.5" y1="41" x2="18" y2="41.5" width="0.254" layer="16"/>
-<wire x1="18" y1="41.5" x2="15" y2="41.5" width="0.254" layer="16"/>
-<via x="15" y="41.5" extent="1-16" drill="0.8" diameter="1.6"/>
-<wire x1="15" y1="41.5" x2="15" y2="44" width="0.6096" layer="1"/>
-<wire x1="15" y1="44" x2="16" y2="45" width="0.6096" layer="1"/>
-<wire x1="16" y1="45" x2="19.73" y2="45" width="0.6096" layer="1"/>
-<wire x1="9" y1="31.5" x2="9" y2="39" width="0.6096" layer="16"/>
-<wire x1="9" y1="39" x2="11.5" y2="41.5" width="0.6096" layer="16"/>
-<wire x1="11.5" y1="41.5" x2="15" y2="41.5" width="0.6096" layer="16"/>
+<via x="7" y="28.5" extent="1-16" drill="0.8" diameter="1.6"/>
+<wire x1="9" y1="31.5" x2="9" y2="42.5" width="0.6096" layer="16"/>
 <wire x1="38.5" y1="26" x2="42" y2="26" width="0.4064" layer="16"/>
-<wire x1="20.5" y1="25" x2="20.5" y2="24" width="0.254" layer="16"/>
+<wire x1="20.5" y1="25" x2="20.5" y2="24" width="0.4064" layer="16"/>
+<wire x1="9" y1="42.5" x2="11.5" y2="45" width="0.6096" layer="16"/>
+<wire x1="11.5" y1="45" x2="19.73" y2="45" width="0.6096" layer="16"/>
+<wire x1="9" y1="28.5" x2="7" y2="28.5" width="0.6096" layer="16"/>
+<wire x1="18" y1="29.525" x2="18" y2="27" width="0.254" layer="16"/>
+<via x="18" y="27" extent="1-16" drill="0.8" diameter="1.6"/>
+<wire x1="21.5" y1="26" x2="19" y2="26" width="0.4064" layer="16"/>
+<wire x1="19" y1="26" x2="18" y2="27" width="0.4064" layer="16"/>
+<wire x1="18" y1="27" x2="16.5" y2="28.5" width="0.6096" layer="1"/>
+<wire x1="16.5" y1="28.5" x2="7" y2="28.5" width="0.6096" layer="1"/>
+<wire x1="3.77" y1="26.29" x2="5.98" y2="28.5" width="0.6096" layer="1"/>
+<wire x1="5.98" y1="28.5" x2="7" y2="28.5" width="0.6096" layer="1"/>
 </signal>
 <signal name="XTAL1">
@@
 <contactref element="Q1" pad="2"/>
 <contactref element="C6" pad="2"/>
-<wire x1="35.7418" y1="21.7434" x2="47.7434" y2="21.7434" width="0.4064" layer="16"/>
 <wire x1="55" y1="27.5" x2="53.5" y2="27.5" width="0.4064" layer="16"/>
-<wire x1="53.5" y1="27.5" x2="47.7434" y2="21.7434" width="0.4064" layer="16"/>
 <wire x1="55" y1="30.5" x2="55" y2="27.5" width="0.6096" layer="16"/>
 <via x="55" y="30.5" extent="1-16" drill="0.8" diameter="1.6"/>
 <wire x1="55" y1="30.5" x2="59.337" y2="26.163" width="0.6096" layer="1"/>
 <wire x1="59.337" y1="26.163" x2="60.5" y2="26.163" width="0.6096" layer="1"/>
+<wire x1="35.7418" y1="21.7434" x2="47.7434" y2="21.7434" width="0.4064" layer="16"/>
+<wire x1="47.7434" y1="21.7434" x2="53.5" y2="27.5" width="0.4064" layer="16"/>
 </signal>
 <signal name="XTAL2">
@@
 <contactref element="Q1" pad="1"/>
 <contactref element="C5" pad="2"/>
-<wire x1="55.5" y1="20" x2="55" y2="20" width="0.6096" layer="16"/>
-<wire x1="35.7418" y1="20.956" x2="37.544" y2="20.956" width="0.4064" layer="16"/>
-<wire x1="37.544" y1="20.956" x2="38.5" y2="20" width="0.4064" layer="16"/>
-<wire x1="38.5" y1="20" x2="55.5" y2="20" width="0.4064" layer="16"/>
-<wire x1="55" y1="17" x2="55" y2="19.5" width="0.6096" layer="16"/>
-<wire x1="55" y1="19.5" x2="55.5" y2="20" width="0.6096" layer="16"/>
+<wire x1="35.7418" y1="20.956" x2="38.044" y2="20.956" width="0.4064" layer="16"/>
+<wire x1="38.044" y1="20.956" x2="39" y2="20" width="0.4064" layer="16"/>
+<wire x1="39" y1="20" x2="41.804115625" y2="20" width="0.4064" layer="16"/>
+<wire x1="41.804115625" y1="20" x2="42.261315625" y2="19.5428" width="0.4064" layer="16" curve="-90"/>
+<wire x1="42.261315625" y1="19.5428" x2="42.261315625" y2="19.0705" width="0.4064" layer="16"/>
+<wire x1="42.261315625" y1="19.0705" x2="42.718515625" y2="18.6133" width="0.4064" layer="16" curve="90"/>
+<wire x1="42.718515625" y1="18.6133" x2="45.0856" y2="18.6133" width="0.4064" layer="16"/>
+<wire x1="45.0856" y1="18.6133" x2="45.5428" y2="19.0705" width="0.4064" layer="16" curve="90"/>
+<wire x1="45.5428" y1="19.0705" x2="45.5428" y2="19.5428" width="0.4064" layer="16"/>
+<wire x1="45.5428" y1="19.5428" x2="46" y2="20" width="0.4064" layer="16" curve="-90"/>
+<wire x1="46" y1="20" x2="55" y2="20" width="0.4064" layer="16"/>
 <via x="55" y="17" extent="1-16" drill="0.8" diameter="1.6"/>
 <wire x1="55" y1="17" x2="59.337" y2="21.337" width="0.6096" layer="1"/>
 <wire x1="59.337" y1="21.337" x2="60.5" y2="21.337" width="0.6096" layer="1"/>
+<wire x1="55" y1="17" x2="55" y2="20" width="0.6096" layer="16"/>
 </signal>
 <signal name="MISO">
@@
 <wire x1="12" y1="16.4" x2="12" y2="22" width="0.6096" layer="16"/>
 <via x="12" y="22" extent="1-16" drill="0.8" diameter="1.6"/>
-<wire x1="3.77" y1="23.75" x2="5.75" y2="23.75" width="0.6096" layer="1"/>
-<wire x1="5.75" y1="23.75" x2="7.5" y2="22" width="0.6096" layer="1"/>
-<wire x1="7.5" y1="22" x2="12" y2="22" width="0.6096" layer="1"/>
+<wire x1="3.77" y1="23.75" x2="4.75" y2="23.75" width="0.6096" layer="1"/>
+<wire x1="4.75" y1="23.75" x2="6.5" y2="22" width="0.6096" layer="1"/>
+<wire x1="6.5" y1="22" x2="12" y2="22" width="0.6096" layer="1"/>
 <wire x1="23" y1="12" x2="22" y2="12" width="0.6096" layer="1"/>
 <wire x1="22" y1="12" x2="12" y2="22" width="0.6096" layer="1"/>
@@
 <wire x1="31.9064" y1="30.9064" x2="32" y2="31" width="0.4064" layer="16"/>
 <via x="32" y="31" extent="1-16" drill="0.8" diameter="1.6"/>
-<wire x1="32" y1="31" x2="4" y2="31" width="0.6096" layer="1"/>
-<wire x1="4" y1="31" x2="1.23" y2="28.23" width="0.6096" layer="1"/>
-<wire x1="1.23" y1="28.23" x2="1.23" y2="26.29" width="0.6096" layer="1"/>
+<wire x1="32" y1="31" x2="5.94" y2="31" width="0.6096" layer="1"/>
 <wire x1="37" y1="33.55" x2="34.55" y2="33.55" width="0.6096" layer="16"/>
 <wire x1="34.55" y1="33.55" x2="32" y2="31" width="0.6096" layer="16"/>
+<wire x1="1.23" y1="26.29" x2="5.94" y2="31" width="0.6096" layer="1"/>
 </signal>
 <signal name="SS">
@@
 <wire x1="26.5" y1="32.5" x2="25" y2="32.5" width="0.3048" layer="16"/>
 <wire x1="19.75" y1="38" x2="19.75" y2="40.75" width="0.6096" layer="16"/>
-<via x="22" y="41.5" extent="1-16" drill="0.8" diameter="1.6"/>
-<wire x1="22.27" y1="41.77" x2="22.27" y2="45" width="0.6096" layer="1"/>
+<wire x1="22.27" y1="41.77" x2="22.27" y2="45" width="0.6096" layer="16"/>
 <wire x1="19.75" y1="40.75" x2="20.5" y2="41.5" width="0.6096" layer="16"/>
 <wire x1="20.5" y1="41.5" x2="22" y2="41.5" width="0.6096" layer="16"/>
-<wire x1="22.27" y1="41.77" x2="22" y2="41.5" width="0.6096" layer="1"/>
+<wire x1="22.27" y1="41.77" x2="22" y2="41.5" width="0.6096" layer="16"/>
 </signal>
 <signal name="N$1">
